File: kicad/firehose_01_ch1.sch (KiCad schematic (older format))
At the start: 57 parts, among them J1 SMA, U1 MAX2112, U2 MAX19505, U20 MIC2090-1YM5, U3 MGA-68563

Commit message: KiCAD schematic complete
Parts:
- C11, C12, C13, C14: footprint (none) -> footprints:0402
Changed lines of the file:
@@
 EELAYER 25 0
 EELAYER END
-$Descr A 11000 8500
+$Descr USLetter 11000 8500
 encoding utf-8
 Sheet 2 10
@@
 F 0 "R1" V 3400 3450 50  0000 C CNN
 F 1 "86.6" V 3500 3500 50  0000 C CNN
-F 2 "" V 3380 3300 50  0000 C CNN
+F 2 "" V 3380 3300 50  0001 C CNN
 F 3 "" H 3450 3300 50  0000 C CNN
 	1    3450 3300
@@
 F 0 "L2" V 1350 3150 50  0000 C CNN
 F 1 "6 nH" V 1450 3100 50  0000 C CNN
-F 2 "" H 1400 3300 50  0000 C CNN
+F 2 "" H 1400 3300 50  0001 C CNN
 F 3 "" H 1400 3300 50  0000 C CNN
 	1    1400 3300
@@
 F 0 "R3" H 3750 2800 50  0000 C CNN
 F 1 "43.2" H 3750 2900 50  0000 C CNN
-F 2 "" V 3630 3050 50  0000 C CNN
+F 2 "" V 3630 3050 50  0001 C CNN
 F 3 "" H 3700 3050 50  0000 C CNN
 	1    3700 3050
@@
 F 0 "L3" V 3000 2600 50  0000 C CNN
 F 1 "47 nH" V 3100 2550 50  0000 C CNN
-F 2 "" H 3050 2700 50  0000 C CNN
+F 2 "" H 3050 2700 50  0001 C CNN
 F 3 "" H 3050 2700 50  0000 C CNN
 	1    3050 2700
@@
 F 0 "L12" V 900 2600 50  0000 C CNN
 F 1 "47 nH" V 1000 2550 50  0000 C CNN
-F 2 "" H 1000 2750 50  0000 C CNN
+F 2 "" H 1000 2750 50  0001 C CNN
 F 3 "" H 1000 2750 50  0000 C CNN
 	1    1000 2750
@@
 F 0 "R2" V 2250 2250 50  0000 C CNN
 F 1 "5.1k" V 2350 2250 50  0000 C CNN
-F 2 "" V 2230 2450 50  0000 C CNN
+F 2 "" V 2230 2450 50  0001 C CNN
 F 3 "" H 2300 2450 50  0000 C CNN
 	1    2300 2450
@@
 F 0 "C11" H 6500 2500 50  0000 C CNN
 F 1 "47 nF" H 6850 2500 50  0000 C CNN
-F 2 "" H 6650 2450 50  0001 C CNN
+F 2 "footprints:0402" H 6650 2450 50  0001 C CNN
 F 3 "" H 6650 2450 50  0001 C CNN
 	1    6650 2450
@@
 F 0 "C12" H 6500 2650 50  0000 C CNN
 F 1 "47 nF" H 6850 2650 50  0000 C CNN
-F 2 "" H 6650 2600 50  0001 C CNN
+F 2 "footprints:0402" H 6650 2600 50  0001 C CNN
 F 3 "" H 6650 2600 50  0001 C CNN
 	1    6650 2600
@@
 F 0 "C13" H 6500 2900 50  0000 C CNN
 F 1 "47 nF" H 6850 2900 50  0000 C CNN
-F 2 "" H 6650 2850 50  0001 C CNN
+F 2 "footprints:0402" H 6650 2850 50  0001 C CNN
 F 3 "" H 6650 2850 50  0001 C CNN
 	1    6650 2850
@@
 F 0 "C14" H 6500 3050 50  0000 C CNN
 F 1 "47 nF" H 6850 3050 50  0000 C CNN
-F 2 "" H 6650 3000 50  0001 C CNN
+F 2 "footprints:0402" H 6650 3000 50  0001 C CNN
 F 3 "" H 6650 3000 50  0001 C CNN
 	1    6650 3000
@@
 F 0 "FB14" H 1400 5650 50  0000 C CNN
 F 1 "240" H 1400 5550 50  0000 C CNN
-F 2 "" H 1450 5750 50  0000 C CNN
+F 2 "" H 1450 5750 50  0001 C CNN
 F 3 "" H 1450 5750 50  0000 C CNN
 	1    1450 5750
@@
 F 0 "R5" V 3750 6050 50  0000 C CNN
 F 1 "390" V 3850 6050 50  0000 C CNN
-F 2 "" V 3680 5900 50  0000 C CNN
+F 2 "" V 3680 5900 50  0001 C CNN
 F 3 "" H 3750 5900 50  0000 C CNN
 	1    3750 5900
@@
 F 0 "R4" H 4050 5500 50  0000 C CNN
 F 1 "820" H 4050 5600 50  0000 C CNN
-F 2 "" V 3980 5750 50  0000 C CNN
+F 2 "" V 3980 5750 50  0001 C CNN
 F 3 "" H 4050 5750 50  0000 C CNN
 	1    4050 5750
@@
 F 0 "R6" H 6500 5900 50  0000 C CNN
 F 1 "10k" H 6300 5900 50  0000 C CNN
-F 2 "" V 6280 5750 50  0000 C CNN
+F 2 "" V 6280 5750 50  0001 C CNN
 F 3 "" H 6350 5750 50  0000 C CNN
 	1    6350 5750
@@
 F 0 "R7" V 8250 6050 50  0000 C CNN
 F 1 "80" V 8350 6050 50  0000 C CNN
-F 2 "" V 8180 5900 50  0000 C CNN
+F 2 "" V 8180 5900 50  0001 C CNN
 F 3 "" H 8250 5900 50  0000 C CNN
 	1    8250 5900
@@
 F 0 "R79" H 5100 6900 50  0000 C CNN
 F 1 "10k" H 4900 6900 50  0000 C CNN
-F 2 "" V 4880 7050 50  0000 C CNN
+F 2 "" V 4880 7050 50  0001 C CNN
 F 3 "" H 4950 7050 50  0000 C CNN
 	1    4950 7050
@@
 F 0 "R80" H 5100 7300 50  0000 C CNN
 F 1 "10k" H 4900 7300 50  0000 C CNN
-F 2 "" V 4880 7400 50  0000 C CNN
+F 2 "" V 4880 7400 50  0001 C CNN
 F 3 "" H 4950 7400 50  0000 C CNN
 	1    4950 7400
@@
 F 0 "FB11" H 1800 6900 50  0000 C CNN
 F 1 "240" H 1800 6800 50  0000 C CNN
-F 2 "" H 1850 7000 50  0000 C CNN
+F 2 "" H 1850 7000 50  0001 C CNN
 F 3 "" H 1850 7000 50  0000 C CNN
 	1    1850 7000

Commit message: footprints and footprint assignments
Parts:
- C1, C10, C15, C16, C17, C18, C19, C20, C21, C22, C23, C24, C242, C243, C25, C26, C27, C28, C29, C30, C31, C32, C33, C34, C35, C36, C37, C5, C6, C7, C8, C9, L12, L2, L3, R1, R2, R3, R4, R5, R6, R7, R79, R80: footprint (none) -> footprints:0402
- FB11, FB14, R126: footprint (none) -> footprints:0603
- J1: footprint (none) -> footprints:SMA_END_LAUNCH
- TP13: footprint (none) -> footprints:TP_SMT
- U1: footprint (none) -> footprints:QFN28_EP
- U2: footprint (none) -> footprints:QFN48_EP
- U20: footprint (none) -> footprints:SOT-23-5
- U3: footprint (none) -> footprints:SOT-363
