File: kicad/firehose_02_ch2.sch (KiCad schematic (older format))
At the start: 0 parts

Commit message: schematic, RF channels 2 and 3
Parts:
- added C100, C81, C82, C91, C92, C93, C94, C95, C96, C97, C98, C99: 0.1 uF, symbol C
- added C244, C245, C83, C84, C85, C86, C87, C88, C89: 1000 pF, symbol C
- added C67, C73, C74, C75, C76, C77: 47 nF, symbol C
- added C68: 10 nF, symbol C
- added C69, C70, C71, C72, C80, C90: 100 pF, symbol C
- added C78: 2.2 nF, symbol C
- added C79: 33 nF, symbol C
- added FB12, FB15: 240, symbol L
- added J2: SMA, symbol SMA
- added L13, L5: 47 nH, symbol L
- added L4: 6 nH, symbol L
- added R127: 0, symbol R
- added R17: 86.6, symbol R
- added R18: 5.1k, symbol R
- added R19: 43.2, symbol R
- added R20: 820, symbol R
- added R21: 390, symbol R
- added R22, R81, R82: 10k, symbol R
- added R23: 80, symbol R
- added TP14: test_point, symbol test_point
- added U21: MIC2090-1YM5, symbol MIC2090-1YM5
- added U4: MAX2112, symbol MAX2112
- added U5: MAX19505, symbol MAX19505
- added U6: MGA-68563, symbol MGA-68563
Connections:
- net labels added: CH2_CLK, CH2_CLK+, CH2_CLK-, CH2_CS, CH2_D0, CH2_D1, CH2_D2, CH2_D3, CH2_D4, CH2_D5, CH2_D6, CH2_D7, CH2_GC1_FPGA_LPF, CH2_REF+, CH2_SCL, CH2_SCLK, CH2_SDA, CH2_SDIN, GND, VCC_3.3V, ch2_cpout, ch2_gc1_lpf, ch2_vcc, ch2_vcc_lna, ch2_vtune, ch2_xtal
- wire segments 0 -> 99
- no-connect marks 0 -> 12
Other:
- note added: "ADC"
- note added: "LNA"
- note added: "RF channel 2"
- note added: "antenna power\nbias tee"
- note added: "downconverter"
- note added: "loop filter"

Commit message: more KiCAD schematic: power symbols, global nets
Other:
- moved on the sheet: C100, C244, C245, C67, C68, C69, C70, C71, C72, C73, C74, C75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

Commit message: footprints and footprint assignments
Parts:
- C100, C244, C245, C67, C68, C69, C70, C71, C72, C73, C74, C75, C76, C77, C78, C79, C80, C81, C82, C83, C84, C85, C86, C87, C88, C89, C90, C91, C92, C93, C94, C95, C96, C97, C98, C99, L13, L4, L5, R17, R18, R19, R20, R21, R22, R23, R81, R82: footprint (none) -> footprints:0402
- FB12, FB15, R127: footprint (none) -> footprints:0603
- J2: footprint (none) -> footprints:SMA_END_LAUNCH
- TP14: footprint (none) -> footprints:TP_SMT
- U21: footprint (none) -> footprints:SOT-23-5
- U4: footprint (none) -> footprints:QFN28_EP
- U5: footprint (none) -> footprints:QFN48_EP
- U6: footprint (none) -> footprints:SOT-363
