File: kicad/firehose_03_ch3.sch (KiCad schematic (older format))
At the start: 0 parts

Commit message: schematic, RF channels 2 and 3
Parts:
- added C102, C108, C109, C110, C111, C112: 47 nF, symbol C
- added C103: 10 nF, symbol C
- added C104, C105, C106, C107, C115, C125: 100 pF, symbol C
- added C113: 2.2 nF, symbol C
- added C114: 33 nF, symbol C
- added C116, C117, C126, C127, C128, C129, C130, C131, C132, C133, C134, C135: 0.1 uF, symbol C
- added C118, C119, C120, C121, C122, C123, C124, C246, C247: 1000 pF, symbol C
- added FB13, FB16: 240, symbol L
- added J3: SMA, symbol SMA
- added L14, L7: 47 nH, symbol L
- added L6: 6 nH, symbol L
- added R128: 0, symbol R
- added R25: 86.6, symbol R
- added R26: 5.1k, symbol R
- added R27: 43.2, symbol R
- added R28: 820, symbol R
- added R29: 390, symbol R
- added R30, R83, R84: 10k, symbol R
- added R31: 80, symbol R
- added TP15: test_point, symbol test_point
- added U22: MIC2090-1YM5, symbol MIC2090-1YM5
- added U7: MAX2112, symbol MAX2112
- added U9: MGA-68563, symbol MGA-68563
- added U?: MAX19505, symbol MAX19505
Connections:
- net labels added: CH3_CLK, CH3_CLK+, CH3_CLK-, CH3_CS, CH3_D0, CH3_D1, CH3_D2, CH3_D3, CH3_D4, CH3_D5, CH3_D6, CH3_D7, CH3_GC1_FPGA_LPF, CH3_REF+, CH3_SCL, CH3_SCLK, CH3_SDA, CH3_SDIN, GND, VCC_3.3V, ch3_cpout, ch3_gc1_lpf, ch3_vcc, ch3_vcc_lna, ch3_vtune, ch3_xtal
- wire segments 0 -> 99
- no-connect marks 0 -> 12
Other:
- note added: "ADC"
- note added: "LNA"
- note added: "RF channel 3"
- note added: "antenna power\nbias tee"
- note added: "downconverter"
- note added: "loop filter"

Commit message: more KiCAD schematic: power symbols, global nets
Parts:
- gave numbers to parts that had none: 1
Other:
- moved on the sheet: C102, C103, C104, C105, C106, C107, C108, C109, C110, C111, C112, C113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

Commit message: footprints and footprint assignments
Parts:
- C102, C103, C104, C105, C106, C107, C108, C109, C110, C111, C112, C113, C114, C115, C116, C117, C118, C119, C120, C121, C122, C123, C124, C125, C126, C127, C128, C129, C130, C131, C132, C133, C134, C135, C246, C247, L14, L6, L7, R25, R26, R27, R28, R29, R30, R31, R83, R84: footprint (none) -> footprints:0402
- FB13, FB16, R128: footprint (none) -> footprints:0603
- J3: footprint (none) -> footprints:SMA_END_LAUNCH
- TP15: footprint (none) -> footprints:TP_SMT
- U22: footprint (none) -> footprints:SOT-23-5
- U7: footprint (none) -> footprints:QFN28_EP
- U8: footprint (none) -> footprints:QFN48_EP
- U9: footprint (none) -> footprints:SOT-363
