File: kicad/firehose_04_ch4.sch (KiCad schematic (older format))
At the start: 0 parts

Commit message: more schematic
Parts:
- added C137, C138, C139, C140, C201, C202, C203, C204, C205, C206, C41, C42, C43: 0.1 uF, symbol C
- added C238, C239, C240, C241: NONE, symbol C
- added J4, J5: SMA, symbol SMA
- added L20, L21: 0, symbol L
- added R129, R130: NONE, symbol R
- added R131, R135, R136: 0, symbol R
- added R33, R37: 49.9, symbol R
- added R34, R35: 60.4, symbol R
- added R36: 249, symbol R
- added U10: MAX19505, symbol MAX19505
Connections:
- net labels added: 10_MHz+, 10_MHz-, CH4_CLK, CH4_CLK+, CH4_CLK-, CH4_CS, CH4_D0, CH4_D1, CH4_D2, CH4_D3, CH4_D4, CH4_D5, CH4_D6, CH4_D7, CH4_SCLK, CH4_SDIN, GND, PPS+, PPS-, VCC_3.3V
- wire segments 0 -> 78
- no-connect marks 0 -> 11
Other:
- note added: "ADC"
- note added: "optional LPF"
- note added: "optional pad"
- note added: "optional\nAC coupling"

Commit message: more KiCAD schematic: power symbols, global nets
Connections:
- wire segments 78 -> 54

Commit message: KiCAD schematic complete
Other:
- moved on the sheet: C137, C138, C139, C140, C201, C202, C203, C204, C205, C206, C238, C239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

Commit message: footprints and footprint assignments
Parts:
- C137, C138, C139, C140, C201, C202, C203, C204, C205, C206, C238, C239, C240, C241, C41, C42, C43, R129, R130, R131, R135, R136, R33, R34, R35, R36, R37: footprint (none) -> footprints:0402
- J4, J5: footprint (none) -> footprints:SMA_END_LAUNCH
- L20, L21: footprint (none) -> footprints:0603
- U10: footprint (none) -> footprints:QFN48_EP
