File: kicad/GNSS_Firehose.sch (KiCad schematic (older format))
At the start: 0 parts

Commit message: more KiCAD schematic
Other:
- note added: "GNSS Firehose"
- note added: "Wideband front end for GPS, GLONASS, Galileo, BeiDou"
Changed lines of the file:
@@
 $Descr A 11000 8500
 encoding utf-8
-Sheet 1 2
+Sheet 1 10
 Title ""
 Date ""
@@
 $EndDescr
 $Sheet
-S 1500 7000 650  550
+S 600  6500 650  550
 U 58CB876E
 F0 "RF channel 1" 60
 F1 "firehose_01_ch1.sch" 60
 $EndSheet
+$Sheet
+S 1950 6600 800  450
+U 58CEAC80
+F0 "RF Channel 2" 60
+F1 "firehose_02_ch2.sch" 60
+$EndSheet
+Text Notes 4400 1400 0    200  ~ 40
+GNSS Firehose
+Text Notes 2550 1950 0    150  ~ 0
+Wideband front end for GPS, GLONASS, Galileo, BeiDou
+$Sheet
+S 3250 6600 800  450
+U 58CEAC97
+F0 "RF Channel 3" 60
+F1 "firehose_03_ch3.sch" 60
+$EndSheet
+$Sheet
+S 4600 6600 800  450
+U 58CEAC9A
+F0 "RF Channel 4" 60
+F1 "firehose_04_ch4.sch" 60
+$EndSheet
+$Sheet
+S 6000 6600 750  450
+U 58CEAC9D
+F0 "Clock generation" 60
+F1 "firehose_05_clock.sch" 60
+$EndSheet
+$Sheet
+S 8800 6600 750  450
+U 58CEACA4
+F0 "Ethernet" 60
+F1 "firehose_07_ethernet.sch" 60
+$EndSheet
+$Sheet
+S 600  7400 750  450
+U 58CEACA7
+F0 "Power" 60
+F1 "firehose_08_power.sch" 60
+$EndSheet
+$Sheet
+S 2050 7400 750  450
+U 58CEACAA
+F0 "Mechanical" 60
+F1 "firehose_09_mechanical.sch" 60
+$EndSheet
+$Sheet
+S 7400 6600 800  450
+U 58CEAF28
+F0 "FPGA" 60
+F1 "firehose_06_fpga.sch" 60
+$EndSheet
 $EndSCHEMATC

Commit message: CAM outputs: position file, BOM
Other:
- note added: "placeholder for\nblock-diagram graphics"
Changed lines of the file:
@@
 $EndDescr
 $Sheet
-S 600  6500 650  550
+S 600  6600 750  450
 U 58CB876E
 F0 "RF channel 1" 60
@@
 $EndSheet
 $Sheet
-S 1950 6600 800  450
+S 1900 6600 750  450
 U 58CEAC80
 F0 "RF Channel 2" 60
 F1 "firehose_02_ch2.sch" 60
 $EndSheet
-Text Notes 4400 1400 0    200  ~ 40
+Text Notes 4250 1400 0    250  ~ 50
 GNSS Firehose
-Text Notes 2550 1950 0    150  ~ 0
+Text Notes 2400 1950 0    150  ~ 30
 Wideband front end for GPS, GLONASS, Galileo, BeiDou
 $Sheet
-S 3250 6600 800  450
+S 3200 6600 750  450
 U 58CEAC97
 F0 "RF Channel 3" 60
@@
 $EndSheet
 $Sheet
-S 4600 6600 800  450
+S 4500 6600 750  450
 U 58CEAC9A
 F0 "RF Channel 4" 60
@@
 $EndSheet
 $Sheet
-S 6000 6600 750  450
+S 5800 6600 750  450
 U 58CEAC9D
 F0 "Clock generation" 60
@@
 $EndSheet
 $Sheet
-S 8800 6600 750  450
+S 8400 6600 750  450
 U 58CEACA4
 F0 "Ethernet" 60
@@
 $EndSheet
 $Sheet
-S 2050 7400 750  450
+S 1900 7400 750  450
 U 58CEACAA
 F0 "Mechanical" 60
@@
 $EndSheet
 $Sheet
-S 7400 6600 800  450
+S 7100 6600 750  450
 U 58CEAF28
 F0 "FPGA" 60
 F1 "firehose_06_fpga.sch" 60
 $EndSheet
+Text Notes 4750 4050 0    100  ~ 0
+placeholder for\nblock-diagram graphics
+Wire Notes Line
+	4150 3100 7050 3100
+Wire Notes Line
+	7050 3100 7050 4900
+Wire Notes Line
+	7050 4900 4150 4900
+Wire Notes Line
+	4150 4900 4150 3100
 $EndSCHEMATC
