File: kicad/firehose_05_clock.sch (KiCad schematic (older format))
At the start: 0 parts

Commit message: more schematic
Parts:
- added OSC?: TCXO, symbol TCXO
- added U?: CDCLVC1102, symbol CDCLVC1102
- added U?: LMK03806, symbol LMK03806
Changed lines of the file:
@@
 EESchema Schematic File Version 2
 LIBS:GNSS_Firehose
+LIBS:GNSS_Firehose-cache
 EELAYER 25 0
 EELAYER END
-$Descr A4 11693 8268
+$Descr A 11000 8500
 encoding utf-8
-Sheet 1 10
+Sheet 6 10
 Title ""
 Date ""
@@
 Comment4 ""
 $EndDescr
+$Comp
+L TCXO OSC?
+U 1 1 58D1264E
+P 1300 3100
+F 0 "OSC?" H 1850 2800 60  0000 C CNN
+F 1 "TCXO" H 1850 2700 60  0000 C CNN
+F 2 "" H 1300 3100 60  0001 C CNN
+F 3 "" H 1300 3100 60  0001 C CNN
+	1    1300 3100
+	1    0    0    -1
+$EndComp
+$Comp
+L CDCLVC1102 U?
+U 1 1 58D12665
+P 3250 3200
+F 0 "U?" H 3700 2750 60  0000 C CNN
+F 1 "CDCLVC1102" H 3900 2600 60  0000 C CNN
+F 2 "" H 3250 3250 60  0001 C CNN
+F 3 "" H 3250 3250 60  0001 C CNN
+	1    3250 3200
+	1    0    0    -1
+$EndComp
+$Comp
+L LMK03806 U?
+U 1 1 58D126BC
+P 8150 3250
+F 0 "U?" H 8050 700 60  0000 C CNN
+F 1 "LMK03806" H 8150 550 60  0000 C CNN
+F 2 "" H 7650 3250 60  0001 C CNN
+F 3 "" H 7650 3250 60  0001 C CNN
+	1    8150 3250
+	1    0    0    -1
+$EndComp
 $EndSCHEMATC

Commit message: more schematic
Parts:
- added C210, C211, C212, C229, C230, C254, C44, C45, C46, C47, C49, C51, C53, C54, C55, C56, C57, C58, C59, C60, C61, C62, C63, C64, C65, C66: 0.1 uF, symbol C
- added C214: 220 pF, symbol C
- added C215: 18 nF, symbol C
- added C231, C232, C233, C234, C235, C236, C255: 10 pF, symbol C
- added FB10, FB17, FB4, FB5, FB6, FB7, FB8, FB9: 240, symbol L
- added L15, L17, L19: 56 nH, symbol L
- added R10: 220, symbol R
- added R11, R13, R15: 80, symbol R
- added R132: 0, symbol R
- added R133, R144: 10, symbol R
- added R88: 820, symbol R
- added R9: 150, symbol R
- added TP1, TP10, TP11, TP12, TP16, TP17, TP2, TP27, TP28, TP29, TP3, TP4, TP5, TP6, TP7, TP8, TP9: test_point, symbol test_point
- gave numbers to parts that had none: 3
Connections:
- net labels added: CH1_CLK+, CH1_CLK-, CH1_REF+, CH2_CLK+, CH2_CLK-, CH2_REF+, CH3_CLK+, CH3_CLK-, CH3_REF+, CH4_CLK+, CH4_CLK-, CLOCK_CLK, CLOCK_DATA, CLOCK_FTEST_LD, CLOCK_LE, CLOCK_READBACK, FPGA_CLK+, FPGA_CLK-, GND, VCC_3.3V, ch1_d+, ch2_d+, ch3_d+, clk_3888
- wire segments 0 -> 130
- no-connect marks 0 -> 2
Other:
- note added: "38.88 MHz TCXO"
- note added: "clock buffer"
- note added: "clock synthesizer"

Commit message: more KiCAD schematic: power symbols, global nets
Connections:
- net labels added: CLK_3888
- net labels removed: clk_3888
- wire segments 130 -> 103

Commit message: fix connections
Connections:
- wire segments 103 -> 104
Other:
- moved on the sheet: C255
Changed lines of the file:
@@
 L C C255
 U 1 1 58D153C7
-P 2200 3900
-F 0 "C255" V 1800 3900 50  0000 C CNN
-F 1 "10 pF" V 1900 3900 50  0000 C CNN
-F 2 "" H 2200 3900 50  0001 C CNN
-F 3 "" H 2200 3900 50  0001 C CNN
-	1    2200 3900
+P 2200 3950
+F 0 "C255" V 1800 3950 50  0000 C CNN
+F 1 "10 pF" V 1900 3950 50  0000 C CNN
+F 2 "" H 2200 3950 50  0001 C CNN
+F 3 "" H 2200 3950 50  0001 C CNN
+	1    2200 3950
 	0    1    1    0
 $EndComp
@@
 L GND #PWR0125
 U 1 1 58D154EC
-P 2200 4100
-F 0 "#PWR0125" H 2400 4000 50  0001 C CNN
-F 1 "GND" H 2400 3900 50  0001 C CNN
-F 2 "" H 2200 4100 50  0001 C CNN
-F 3 "" H 2200 4100 50  0001 C CNN
-	1    2200 4100
+P 2200 4150
+F 0 "#PWR0125" H 2400 4050 50  0001 C CNN
+F 1 "GND" H 2400 3950 50  0001 C CNN
+F 2 "" H 2200 4150 50  0001 C CNN
+F 3 "" H 2200 4150 50  0001 C CNN
+	1    2200 4150
 	1    0    0    -1
 $EndComp
@@
 Wire Wire Line
 	1900 7400 1900 7300
-Wire Wire Line
-	6700 7000 9350 7000
 Wire Wire Line
 	6800 4350 6250 4350
@@
 Wire Wire Line
 	8700 5950 9150 5950
+Wire Wire Line
+	2200 3800 2200 3750
+Connection ~ 2200 3750
+Wire Wire Line
+	6700 7000 9350 7000
+Connection ~ 7100 7000
+Connection ~ 7500 7000
+Connection ~ 7900 7000
+Connection ~ 8300 7000
+Connection ~ 8700 7000
+Connection ~ 9100 7000
 $EndSCHEMATC

Commit message: footprints and footprint assignments
Parts:
- C210, C211, C212, C214, C229, C230, C231, C232, C233, C234, C235, C236, C254, C255, C44, C45, C46, C47, C49, C51, C54, C55, C56, C57, C58, C59, C60, C61, C62, C63, C64, C65, C66, FB10, FB17, FB4, FB5, FB6, FB7, FB8, FB9, R10, R11, R13, R144, R15, R88, R9: footprint (none) -> footprints:0402
- C215, L15, L17, L19, R132, R133: footprint (none) -> footprints:0603
- C53: value 0.1 uF -> 10 uF; footprint (none) -> footprints:0805
- OSC1: footprint (none) -> footprints:D75J
- TP1, TP10, TP11, TP12, TP16, TP17, TP2, TP27, TP28, TP29, TP3, TP4, TP5, TP6, TP7, TP8, TP9: footprint (none) -> footprints:TP_SMT
- U15: footprint (none) -> footprints:LLP64_EP
- U19: footprint (none) -> footprints:TSSOP8W

Commit message: add page titles to schematic
Other:
- note added: "Clock"
Changed lines of the file:
@@
 	1    0    0    -1
 $EndComp
+Text Notes 9400 900  0    150  ~ 30
+Clock
 $EndSCHEMATC
