File: kicad/firehose_06_fpga.sch (KiCad schematic (older format))
At the start: 0 parts

Commit message: more schematic
Parts:
- added U? (x3): XC6SLX9-2TQG144C, symbol XC6SLX9-2TQG144C
Changed lines of the file:
@@
 EELAYER 25 0
 EELAYER END
-$Descr A4 11693 8268
+$Descr USLetter 11000 8500
 encoding utf-8
-Sheet 1 10
+Sheet 10 10
 Title ""
 Date ""
@@
 Comment4 ""
 $EndDescr
+$Comp
+L XC6SLX9-2TQG144C U?
+U 1 1 58D2BF46
+P 3000 1600
+F 0 "U?" H 3850 -3200 60  0000 C CNN
+F 1 "XC6SLX9-2TQG144C" H 4150 -3300 60  0000 C CNN
+F 2 "" H 3000 1400 60  0001 C CNN
+F 3 "" H 3000 1400 60  0001 C CNN
+	1    3000 1600
+	1    0    0    -1
+$EndComp
+$Comp
+L XC6SLX9-2TQG144C U?
+U 2 1 58D2BFA5
+P 6600 2900
+F 0 "U?" H 7100 2500 60  0000 C CNN
+F 1 "XC6SLX9-2TQG144C" H 7200 2400 60  0000 C CNN
+F 2 "" H 6600 2700 60  0001 C CNN
+F 3 "" H 6600 2700 60  0001 C CNN
+	2    6600 2900
+	1    0    0    -1
+$EndComp
+$Comp
+L XC6SLX9-2TQG144C U?
+U 3 1 58D2BFE0
+P 6650 5200
+F 0 "U?" H 6750 3400 60  0000 C CNN
+F 1 "XC6SLX9-2TQG144C" H 6750 3300 60  0000 C CNN
+F 2 "" H 6650 5000 60  0001 C CNN
+F 3 "" H 6650 5000 60  0001 C CNN
+	3    6650 5200
+	1    0    0    -1
+$EndComp
 $EndSCHEMATC

Commit message: more schematic
Parts:
- added C141, C143, C144, C145, C146, C147, C149, C150, C151, C152, C153, C155, C156, C157, C159, C160, C161, C163, C164, C165, C167, C168, C207, C208, C209, C248, C249: 0.1 uF, symbol C
- added C142, C148, C154, C158, C162, C166: 10 uF, symbol C
- added J10: HEADER_16, symbol HEADER_16
- added J6: HEADER_14, symbol HEADER_14
- added LED1, LED2, LED3: LED, symbol LED
- added R137, R138, R139, R140, R141, R142, R40, R41, R86: 1k, symbol R
- added R146, R147, R148, R149, R150, R46, R76, R77, R78: 10k, symbol R
- added R38, R39, R43, R48: 47, symbol R
- added R42: 0, symbol R
- added R44, R47: 4.7k, symbol R
- added R45, R49, R50, R85: 330, symbol R
- added TP18, TP19, TP20: test_point, symbol test_point
- added U11: AT25DF041A, symbol AT25DF041A
- gave numbers to parts that had none: 1
Connections:
- net labels added: CH1_CLK, CH1_CS, CH1_D0, CH1_D1, CH1_D2, CH1_D3, CH1_D4, CH1_D5, CH1_D6, CH1_D7, CH1_GC1, CH1_GC1_FPGA_LPF, CH1_SCL, CH1_SCLK, CH1_SDA, CH1_SDIN, CH2_CLK, CH2_CS, CH2_D0, CH2_D1, CH2_D2, CH2_D3, CH2_D4, CH2_D5, CH2_D6, CH2_D7, CH2_GC1, CH2_GC1_FPGA_LPF, CH2_SCL, CH2_SCLK, CH2_SDA, CH2_SDIN, CH3_CLK, CH3_CS, CH3_D0, CH3_D1, CH3_D2, CH3_D3, CH3_D4, CH3_D5, CH3_D6, CH3_D7, CH3_GC1, CH3_GC1_FPGA_LPF, CH3_SCL, CH3_SCLK, CH3_SDA, CH3_SDIN, CH4_CLK, CH4_CS, CH4_D0, CH4_D1, CH4_D2, CH4_D3, CH4_D4, CH4_D5, CH4_D6, CH4_D7, CH4_SCLK, CH4_SDIN, CLOCK_CLK, CLOCK_DATA, CLOCK_FTEST_LD, CLOCK_LE, CLOCK_READBACK, FPGA_CLK+, FPGA_CLK-, GND, PHY_MDC, PHY_MDINT, PHY_MDIO, PHY_NRESET, PHY_RXD0, PHY_RXD1, PHY_RXD2, PHY_RXD3, PHY_RX_CLK, PHY_RX_CTL, PHY_TXD0, PHY_TXD1, PHY_TXD2, PHY_TXD3, PHY_TX_CLK, PHY_TX_CTL, TCK, TDI, TDO, TMS, UART_RX, UART_TX, VCC_1.2V, VCC_3.3V, cclk, clk_3888, cso_b, din, init_b, led0, led1, m0, m1, mosi, spare1_n, spare1_p, spare2_n, spare2_p, spare3_n, spare3_p
- wire segments 0 -> 208
- no-connect marks 0 -> 3

Commit message: more KiCAD schematic: power symbols, global nets
Other:
- moved on the sheet: C248, C249

Commit message: fix 1.2V power symbol and pin name.  Netlists are now identical between gEDA and KiCAD
Changed lines of the file:
@@
 Connection ~ 9000 1700
 $Comp
-L GND #PWR0199
+L GND #PWR235
 U 1 1 58D9A68D
 P 9000 1850
-F 0 "#PWR0199" H 9200 1750 50  0001 C CNN
+F 0 "#PWR235" H 9200 1750 50  0001 C CNN
 F 1 "GND" H 9200 1650 50  0001 C CNN
 F 2 "" H 9000 1850 50  0001 C CNN
@@
 $EndComp
 Wire Wire Line
-	5300 4400 6100 4400
-Wire Wire Line
 	6400 4400 6550 4400
 Wire Wire Line
@@
 CH1_GC1
 $Comp
-L GND #PWR0200
+L GND #PWR213
 U 1 1 58DA3CAD
 P 1000 3550
-F 0 "#PWR0200" H 1200 3450 50  0001 C CNN
+F 0 "#PWR213" H 1200 3450 50  0001 C CNN
 F 1 "GND" H 1200 3350 50  0001 C CNN
 F 2 "" H 1000 3550 50  0001 C CNN
@@
 Connection ~ 6300 5900
 $Comp
-L GND #PWR0201
+L GND #PWR225
 U 1 1 58DA7D1C
 P 6300 6150
-F 0 "#PWR0201" H 6500 6050 50  0001 C CNN
+F 0 "#PWR225" H 6500 6050 50  0001 C CNN
 F 1 "GND" H 6500 5950 50  0001 C CNN
 F 2 "" H 6300 6150 50  0001 C CNN
@@
 	10300 5500 10300 5450
 $Comp
-L GND #PWR0202
+L GND #PWR239
 U 1 1 58DA9CBE
 P 9750 6200
-F 0 "#PWR0202" H 9950 6100 50  0001 C CNN
+F 0 "#PWR239" H 9950 6100 50  0001 C CNN
 F 1 "GND" H 9950 6000 50  0001 C CNN
 F 2 "" H 9750 6200 50  0001 C CNN
@@
 	10050 6650 10050 6700
 $Comp
-L GND #PWR0203
+L GND #PWR241
 U 1 1 58DAF55A
 P 10050 6750
-F 0 "#PWR0203" H 10250 6650 50  0001 C CNN
+F 0 "#PWR241" H 10250 6650 50  0001 C CNN
 F 1 "GND" H 10250 6550 50  0001 C CNN
 F 2 "" H 10050 6750 50  0001 C CNN
@@
 $EndComp
 $Comp
-L GND #PWR0204
+L GND #PWR242
 U 1 1 58DAF5D1
 P 10050 7100
-F 0 "#PWR0204" H 10250 7000 50  0001 C CNN
+F 0 "#PWR242" H 10250 7000 50  0001 C CNN
 F 1 "GND" H 10250 6900 50  0001 C CNN
 F 2 "" H 10050 7100 50  0001 C CNN
@@
 init_b
 $Comp
-L GND #PWR0205
+L GND #PWR229
 U 1 1 58DB0C9A
 P 7400 3750
-F 0 "#PWR0205" H 7600 3650 50  0001 C CNN
+F 0 "#PWR229" H 7600 3650 50  0001 C CNN
 F 1 "GND" H 7600 3550 50  0001 C CNN
 F 2 "" H 7400 3750 50  0001 C CNN
@@
 $EndComp
 $Comp
-L GND #PWR0206
+L GND #PWR236
 U 1 1 58DB21F9
 P 9150 2400
-F 0 "#PWR0206" H 9350 2300 50  0001 C CNN
+F 0 "#PWR236" H 9350 2300 50  0001 C CNN
 F 1 "GND" H 9350 2200 50  0001 C CNN
 F 2 "" H 9150 2400 50  0001 C CNN
@@
 TDI
 $Comp
-L GND #PWR0207
+L GND #PWR226
 U 1 1 58DB429B
 P 7400 1050
-F 0 "#PWR0207" H 7600 950 50  0001 C CNN
+F 0 "#PWR226" H 7600 950 50  0001 C CNN
 F 1 "GND" H 7600 850 50  0001 C CNN
 F 2 "" H 7400 1050 50  0001 C CNN
@@
 $EndComp
 $Comp
-L GND #PWR0208
+L GND #PWR227
 U 1 1 58DB48D4
 P 7400 1550
-F 0 "#PWR0208" H 7600 1450 50  0001 C CNN
+F 0 "#PWR227" H 7600 1450 50  0001 C CNN
 F 1 "GND" H 7600 1350 50  0001 C CNN
 F 2 "" H 7400 1550 50  0001 C CNN
@@
 $EndComp
 $Comp
-L GND #PWR0209
+L GND #PWR228
 U 1 1 58DB49DB
 P 7400 2050
-F 0 "#PWR0209" H 7600 1950 50  0001 C CNN
+F 0 "#PWR228" H 7600 1950 50  0001 C CNN
 F 1 "GND" H 7600 1850 50  0001 C CNN
 F 2 "" H 7400 2050 50  0001 C CNN
@@
 	8650 4000 8650 4500
 $Comp
-L GND #PWR0210
+L GND #PWR234
 U 1 1 58DB5863
 P 8650 4550
-F 0 "#PWR0210" H 8850 4450 50  0001 C CNN
+F 0 "#PWR234" H 8850 4450 50  0001 C CNN
 F 1 "GND" H 8850 4350 50  0001 C CNN
 F 2 "" H 8650 4550 50  0001 C CNN
@@
 	9650 4000 9650 4500
 $Comp
-L GND #PWR0211
+L GND #PWR238
 U 1 1 58DB5C46
 P 9650 4550
-F 0 "#PWR0211" H 9850 4450 50  0001 C CNN
+F 0 "#PWR238" H 9850 4450 50  0001 C CNN
 F 1 "GND" H 9850 4350 50  0001 C CNN
 F 2 "" H 9650 4550 50  0001 C CNN
@@
 	10000 3500 10250 3500
 $Comp
-L GND #PWR0212
+L GND #PWR244
 U 1 1 58DB8BB7
 P 10250 3550
-F 0 "#PWR0212" H 10450 3450 50  0001 C CNN
+F 0 "#PWR244" H 10450 3450 50  0001 C CNN
 F 1 "GND" H 10450 3350 50  0001 C CNN
 F 2 "" H 10250 3550 50  0001 C CNN
@@
 Connection ~ 3800 7800
 $Comp
-L GND #PWR0213
+L GND #PWR214
 U 1 1 58DC0219
 P 2550 7150
-F 0 "#PWR0213" H 2750 7050 50  0001 C CNN
+F 0 "#PWR214" H 2750 7050 50  0001 C CNN
 F 1 "GND" H 2750 6950 50  0001 C CNN
 F 2 "" H 2550 7150 50  0001 C CNN
@@
 $EndComp
 $Comp
-L GND #PWR0214
+L GND #PWR215
 U 1 1 58DC042A
 P 2550 7850
-F 0 "#PWR0214" H 2750 7750 50  0001 C CNN
+F 0 "#PWR215" H 2750 7750 50  0001 C CNN
 F 1 "GND" H 2750 7650 50  0001 C CNN
 F 2 "" H 2550 7850 50  0001 C CNN
@@
 $EndComp
 $Comp
-L GND #PWR0215
+L GND #PWR218
 U 1 1 58DC0513
 P 4000 7150
-F 0 "#PWR0215" H 4200 7050 50  0001 C CNN
+F 0 "#PWR218" H 4200 7050 50  0001 C CNN
 F 1 "GND" H 4200 6950 50  0001 C CNN
 F 2 "" H 4000 7150 50  0001 C CNN
@@
 $EndComp
 $Comp
-L GND #PWR0216
+L GND #PWR219
 U 1 1 58DC05FC
 P 4000 7850
-F 0 "#PWR0216" H 4200 7750 50  0001 C CNN
+F 0 "#PWR219" H 4200 7750 50  0001 C CNN
 F 1 "GND" H 4200 7650 50  0001 C CNN
 F 2 "" H 4000 7850 50  0001 C CNN
@@
 Connection ~ 5350 7800
 $Comp
-L GND #PWR0217
+L GND #PWR222
 U 1 1 58DC1ED9
 P 5550 7150
-F 0 "#PWR0217" H 5750 7050 50  0001 C CNN
+F 0 "#PWR222" H 5750 7050 50  0001 C CNN
 F 1 "GND" H 5750 6950 50  0001 C CNN
 F 2 "" H 5550 7150 50  0001 C CNN
@@
 $EndComp
 $Comp
-L GND #PWR0218
+L GND #PWR223
 U 1 1 58DC1FC2
 P 5550 7850
-F 0 "#PWR0218" H 5750 7750 50  0001 C CNN
+F 0 "#PWR223" H 5750 7750 50  0001 C CNN
 F 1 "GND" H 5750 7650 50  0001 C CNN
 F 2 "" H 5550 7850 50  0001 C CNN
@@
 $EndComp
 $Comp
-L VCC_1.2V #PWR0219
-U 1 1 58DEC191
-P 650 6800
-F 0 "#PWR0219" H 830 6570 50  0001 C CNN
-F 1 "VCC_1.2V" H 780 6670 50  0001 C CNN
-F 2 "" H 650 6800 50  0001 C CNN
-F 3 "" H 650 6800 50  0001 C CNN
-	1    650  6800
-	1    0    0    -1
-$EndComp
-$Comp
-L VCC_3.3V #PWR0220
+L VCC_3.3V #PWR212
 U 1 1 58DEC239
 P 650 7500
-F 0 "#PWR0220" H 830 7270 50  0001 C CNN
+F 0 "#PWR212" H 830 7270 50  0001 C CNN
 F 1 "VCC_3.3V" H 780 7370 50  0001 C CNN
 F 2 "" H 650 7500 50  0001 C CNN
@@
 	650  6800 2350 6800
 $Comp
-L VCC_3.3V #PWR0221
+L VCC_3.3V #PWR216
 U 1 1 58DED318
 P 2650 6800
-F 0 "#PWR0221" H 2830 6570 50  0001 C CNN
+F 0 "#PWR216" H 2830 6570 50  0001 C CNN
 F 1 "VCC_3.3V" H 2780 6670 50  0001 C CNN
 F 2 "" H 2650 6800 50  0001 C CNN
@@
 $EndComp
 $Comp
-L VCC_3.3V #PWR0222
+L VCC_3.3V #PWR217
 U 1 1 58DED401
 P 2650 7500
-F 0 "#PWR0222" H 2830 7270 50  0001 C CNN
+F 0 "#PWR217" H 2830 7270 50  0001 C CNN
 F 1 "VCC_3.3V" H 2780 7370 50  0001 C CNN
 F 2 "" H 2650 7500 50  0001 C CNN
@@
 $EndComp
 $Comp
-L VCC_3.3V #PWR0223
+L VCC_3.3V #PWR220
 U 1 1 58DED4EA
 P 4200 6800
-F 0 "#PWR0223" H 4380 6570 50  0001 C CNN
+F 0 "#PWR220" H 4380 6570 50  0001 C CNN
 F 1 "VCC_3.3V" H 4330 6670 50  0001 C CNN
 F 2 "" H 4200 6800 50  0001 C CNN
@@
 $EndComp
 $Comp
-L VCC_3.3V #PWR0224
+L VCC_3.3V #PWR221
 U 1 1 58DED5D3
 P 4200 7500
-F 0 "#PWR0224" H 4380 7270 50  0001 C CNN
+F 0 "#PWR221" H 4380 7270 50  0001 C CNN
 F 1 "VCC_3.3V" H 4330 7370 50  0001 C CNN
 F 2 "" H 4200 7500 50  0001 C CNN
@@
 	4200 7500 5350 7500
 $Comp
-L VCC_1.2V #PWR0225
-U 1 1 58DEFB42
-P 6000 6800
-F 0 "#PWR0225" H 6180 6570 50  0001 C CNN
-F 1 "VCC_1.2V" H 6130 6670 50  0001 C CNN
-F 2 "" H 6000 6800 50  0001 C CNN
-F 3 "" H 6000 6800 50  0001 C CNN
-	1    6000 6800
-	1    0    0    -1
-$EndComp
-$Comp
-L VCC_3.3V #PWR0226
+L VCC_3.3V #PWR232
 U 1 1 58DEFC2B
 P 8100 6900
-F 0 "#PWR0226" H 8280 6670 50  0001 C CNN
+F 0 "#PWR232" H 8280 6670 50  0001 C CNN
 F 1 "VCC_3.3V" H 8230 6770 50  0001 C CNN
 F 2 "" H 8100 6900 50  0001 C CNN
@@
 $EndComp
 $Comp
-L VCC_3.3V #PWR0227
+L VCC_3.3V #PWR233
 U 1 1 58DEFD14
 P 8600 5050
-F 0 "#PWR0227" H 8780 4820 50  0001 C CNN
+F 0 "#PWR233" H 8780 4820 50  0001 C CNN
 F 1 "VCC_3.3V" H 8730 4920 50  0001 C CNN
 F 2 "" H 8600 5050 50  0001 C CNN
@@
 $EndComp
 $Comp
-L VCC_3.3V #PWR0228
+L VCC_3.3V #PWR230
 U 1 1 58DEFDFD
 P 7650 3500
-F 0 "#PWR0228" H 7830 3270 50  0001 C CNN
+F 0 "#PWR230" H 7830 3270 50  0001 C CNN
 F 1 "VCC_3.3V" H 7780 3370 50  0001 C CNN
 F 2 "" H 7650 3500 50  0001 C CNN
@@
 $EndComp
 $Comp
-L VCC_3.3V #PWR0229
+L VCC_3.3V #PWR231
 U 1 1 58DEFEE6
 P 7650 3900
-F 0 "#PWR0229" H 7830 3670 50  0001 C CNN
+F 0 "#PWR231" H 7830 3670 50  0001 C CNN
 F 1 "VCC_3.3V" H 7780 3770 50  0001 C CNN
 F 2 "" H 7650 3900 50  0001 C CNN
@@
 $EndComp
 $Comp
-L VCC_3.3V #PWR0230
+L VCC_3.3V #PWR237
 U 1 1 58DEFFCF
 P 9550 3150
-F 0 "#PWR0230" H 9730 2920 50  0001 C CNN
+F 0 "#PWR237" H 9730 2920 50  0001 C CNN
 F 1 "VCC_3.3V" H 9680 3020 50  0001 C CNN
 F 2 "" H 9550 3150 50  0001 C CNN
@@
 $EndComp
 $Comp
-L VCC_3.3V #PWR0231
+L VCC_3.3V #PWR243
 U 1 1 58DF00B8
 P 10200 2700
-F 0 "#PWR0231" H 10380 2470 50  0001 C CNN
+F 0 "#PWR243" H 10380 2470 50  0001 C CNN
 F 1 "VCC_3.3V" H 10330 2570 50  0001 C CNN
 F 2 "" H 10200 2700 50  0001 C CNN
@@
 $EndComp
 $Comp
-L VCC_3.3V #PWR0232
+L VCC_3.3V #PWR240
 U 1 1 58DF01A1
 P 9900 1100
-F 0 "#PWR0232" H 10080 870 50  0001 C CNN
+F 0 "#PWR240" H 10080 870 50  0001 C CNN
 F 1 "VCC_3.3V" H 10030 970 50  0001 C CNN
 F 2 "" H 9900 1100 50  0001 C CNN
@@
 Text GLabel 5500 6100 2    50   Input ~ 0
 CH4_CLK
+$Comp
+L VCC_1.2V #PWR211
+U 1 1 58DF6752
+P 650 6800
+F 0 "#PWR211" H 830 6570 50  0001 C CNN
+F 1 "VCC_1.2V" H 780 6670 50  0001 C CNN
+F 2 "" H 650 6800 50  0001 C CNN
+F 3 "" H 650 6800 50  0001 C CNN
+	1    650  6800
+	1    0    0    -1
+$EndComp
+$Comp
+L VCC_1.2V #PWR224
+U 1 1 58DF6842
+P 6000 6800
+F 0 "#PWR224" H 6180 6570 50  0001 C CNN
+F 1 "VCC_1.2V" H 6130 6670 50  0001 C CNN
+F 2 "" H 6000 6800 50  0001 C CNN
+F 3 "" H 6000 6800 50  0001 C CNN
+	1    6000 6800
+	1    0    0    -1
+$EndComp
+Wire Wire Line
+	6100 4400 5300 4400
 $EndSCHEMATC

Commit message: footprints and footprint assignments
Parts:
- C141, C143, C144, C145, C146, C147, C149, C150, C151, C152, C153, C155, C156, C157, C159, C160, C161, C163, C164, C165, C167, C168, C207, C208, C209, C248, C249, R137, R138, R139, R140, R141, R142, R146, R147, R148, R149, R150, R38, R39, R40, R41, R42, R43, R44, R45, R46, R47, R48, R49, R50, R76, R77, R78, R85, R86: footprint (none) -> footprints:0402
- C142, C148, C154, C158, C162, C166: footprint (none) -> footprints:0805
- J10: footprint (none) -> footprints:HEADER16_100MIL
- J6: footprint (none) -> footprints:HEADER14_2MM
- LED1: footprint (none) -> footprints:0603
- LED2, LED3: footprint (none) -> footprints:APA2106
- TP18, TP19, TP20: footprint (none) -> footprints:TP_SMT
- U11: footprint (none) -> footprints:SO8
- U12: footprint (none) -> footprints:LQFP144

Commit message: add page titles to schematic
Other:
- note added: "FPGA"
- note added: "JTAG"
- note added: "flash"
Changed lines of the file:
@@
 $Descr USLetter 11000 8500
 encoding utf-8
-Sheet 10 10
+Sheet 7 10
 Title ""
 Date ""
@@
 Wire Wire Line
 	6100 4400 5300 4400
+Text Notes 9250 750  0    150  ~ 30
+FPGA
+Text Notes 10050 2100 0    100  ~ 20
+JTAG
+Text Notes 8800 6150 0    100  ~ 20
+flash
 $EndSCHEMATC
