File: kicad/firehose_07_ethernet.sch (KiCad schematic (older format))
At the start: 0 parts

Commit message: more KiCAD schematic
Parts:
- added C176, C177: 33 pF, symbol C
- added C182, C183, C184, C185, C186, C187, C218, C219, C221, C222, C223, C224, C227, C228, C250, C251, C252, C253: 0.1 uF, symbol C
- added C193, C216, C217, C220, C225, C226: 10 uF, symbol C
- added FB1, FB2, FB3: 240, symbol L
- added J7: L829-1J1T-43, symbol L829-1J1T-43
- added R100, R101, R102, R103, R104, R105: 33, symbol R
- added R106, R109, R110, R113, R118, R119, R123: 1k, symbol R
- added R107: 4.7k, symbol R
- added R108, R111, R112, R114, R115, R120, R121, R122, R125: NONE, symbol R
- added R116, R117, R124, R97: 10k, symbol R
- added R51, R52: 220, symbol R
- added R95: 12.1k 1%, symbol R
- added R96: 470, symbol R
- added R98, R99: 0, symbol R
- added TP22: test_point, symbol test_point
- added U18: KSZ9031RNX, symbol KSZ9031RNX
- added Y1: 25 MHz, symbol crystal
Connections:
- net labels added: AVDDH, AVDDL, AVDDL_PLL, DVDDH, DVDDL, GND, LED_MODE, PHY_MDC, PHY_MDINT, PHY_MDIO, PHY_NRESET, PHY_RXD0, PHY_RXD1, PHY_RXD2, PHY_RXD3, PHY_RX_CLK, PHY_RX_CTL, PHY_TXD0, PHY_TXD1, PHY_TXD2, PHY_TXD3, PHY_TX_CLK, PHY_TX_CTL, VCC_1.2V, VCC_3.3V, chassis_gnd, ct1, ct2, ct3, ct4, phyad0, phyad1, xtal1, xtal2
- wire segments 0 -> 192
- no-connect marks 0 -> 3

Commit message: more KiCAD schematic: power symbols, global nets
Connections:
- wire segments 192 -> 130

Commit message: fix 1.2V power symbol and pin name.  Netlists are now identical between gEDA and KiCAD
Changed lines of the file:
@@
 $EndComp
 $Comp
-L GND #PWR0160
+L GND #PWR166
 U 1 1 58DC9CF5
 P 4100 5600
-F 0 "#PWR0160" H 4300 5500 50  0001 C CNN
+F 0 "#PWR166" H 4300 5500 50  0001 C CNN
 F 1 "GND" H 4300 5400 50  0001 C CNN
 F 2 "" H 4100 5600 50  0001 C CNN
@@
 $EndComp
 $Comp
-L GND #PWR0161
+L GND #PWR164
 U 1 1 58DCAC81
 P 3700 6100
-F 0 "#PWR0161" H 3900 6000 50  0001 C CNN
+F 0 "#PWR164" H 3900 6000 50  0001 C CNN
 F 1 "GND" H 3900 5900 50  0001 C CNN
 F 2 "" H 3700 6100 50  0001 C CNN
@@
 $EndComp
 $Comp
-L GND #PWR0162
+L GND #PWR169
 U 1 1 58DCAD40
 P 5300 6800
-F 0 "#PWR0162" H 5500 6700 50  0001 C CNN
+F 0 "#PWR169" H 5500 6700 50  0001 C CNN
 F 1 "GND" H 5500 6600 50  0001 C CNN
 F 2 "" H 5300 6800 50  0001 C CNN
@@
 $EndComp
 $Comp
-L GND #PWR0163
+L GND #PWR165
 U 1 1 58DCADB7
 P 3700 7300
-F 0 "#PWR0163" H 3900 7200 50  0001 C CNN
+F 0 "#PWR165" H 3900 7200 50  0001 C CNN
 F 1 "GND" H 3900 7100 50  0001 C CNN
 F 2 "" H 3700 7300 50  0001 C CNN
@@
 $EndComp
 $Comp
-L GND #PWR0164
+L GND #PWR163
 U 1 1 58DCAE2E
 P 3300 7800
-F 0 "#PWR0164" H 3500 7700 50  0001 C CNN
+F 0 "#PWR163" H 3500 7700 50  0001 C CNN
 F 1 "GND" H 3500 7600 50  0001 C CNN
 F 2 "" H 3300 7800 50  0001 C CNN
@@
 $EndComp
 $Comp
-L GND #PWR0165
+L GND #PWR167
 U 1 1 58DCD224
 P 4500 4600
-F 0 "#PWR0165" H 4700 4500 50  0001 C CNN
+F 0 "#PWR167" H 4700 4500 50  0001 C CNN
 F 1 "GND" H 4700 4400 50  0001 C CNN
 F 2 "" H 4500 4600 50  0001 C CNN
@@
 $EndComp
 $Comp
-L GND #PWR0166
+L GND #PWR162
 U 1 1 58DCD34F
 P 1800 3500
-F 0 "#PWR0166" H 2000 3400 50  0001 C CNN
+F 0 "#PWR162" H 2000 3400 50  0001 C CNN
 F 1 "GND" H 2000 3300 50  0001 C CNN
 F 2 "" H 1800 3500 50  0001 C CNN
@@
 $EndComp
 $Comp
-L GND #PWR0167
+L GND #PWR171
 U 1 1 58DCD3C6
 P 6200 4400
-F 0 "#PWR0167" H 6400 4300 50  0001 C CNN
+F 0 "#PWR171" H 6400 4300 50  0001 C CNN
 F 1 "GND" H 6400 4200 50  0001 C CNN
 F 2 "" H 6200 4400 50  0001 C CNN
@@
 $EndComp
 $Comp
-L GND #PWR0168
+L GND #PWR168
 U 1 1 58DCD43D
 P 4900 5600
-F 0 "#PWR0168" H 5100 5500 50  0001 C CNN
+F 0 "#PWR168" H 5100 5500 50  0001 C CNN
 F 1 "GND" H 5100 5400 50  0001 C CNN
 F 2 "" H 4900 5600 50  0001 C CNN
@@
 $EndComp
 $Comp
-L GND #PWR0169
+L GND #PWR170
 U 1 1 58DCD4D8
 P 5500 5600
-F 0 "#PWR0169" H 5700 5500 50  0001 C CNN
+F 0 "#PWR170" H 5700 5500 50  0001 C CNN
 F 1 "GND" H 5700 5400 50  0001 C CNN
 F 2 "" H 5500 5600 50  0001 C CNN
@@
 $EndComp
 $Comp
-L GND #PWR0170
+L GND #PWR174
 U 1 1 58DCD54F
 P 7250 4450
-F 0 "#PWR0170" H 7450 4350 50  0001 C CNN
+F 0 "#PWR174" H 7450 4350 50  0001 C CNN
 F 1 "GND" H 7450 4250 50  0001 C CNN
 F 2 "" H 7250 4450 50  0001 C CNN
@@
 $EndComp
 $Comp
-L GND #PWR0171
+L GND #PWR173
 U 1 1 58DD3C92
 P 6850 4450
-F 0 "#PWR0171" H 7050 4350 50  0001 C CNN
+F 0 "#PWR173" H 7050 4350 50  0001 C CNN
 F 1 "GND" H 7050 4250 50  0001 C CNN
 F 2 "" H 6850 4450 50  0001 C CNN
@@
 $EndComp
 $Comp
-L GND #PWR0172
+L GND #PWR179
 U 1 1 58DD3EB4
 P 8050 4450
-F 0 "#PWR0172" H 8250 4350 50  0001 C CNN
+F 0 "#PWR179" H 8250 4350 50  0001 C CNN
 F 1 "GND" H 8250 4250 50  0001 C CNN
 F 2 "" H 8050 4450 50  0001 C CNN
@@
 $EndComp
 $Comp
-L GND #PWR0173
+L GND #PWR176
 U 1 1 58DD3EC2
 P 7650 4450
-F 0 "#PWR0173" H 7850 4350 50  0001 C CNN
+F 0 "#PWR176" H 7850 4350 50  0001 C CNN
 F 1 "GND" H 7850 4250 50  0001 C CNN
 F 2 "" H 7650 4450 50  0001 C CNN
@@
 DVDDH
 $Comp
-L GND #PWR0174
+L GND #PWR180
 U 1 1 58DDA094
 P 9900 6050
-F 0 "#PWR0174" H 10100 5950 50  0001 C CNN
+F 0 "#PWR180" H 10100 5950 50  0001 C CNN
 F 1 "GND" H 10100 5850 50  0001 C CNN
 F 2 "" H 9900 6050 50  0001 C CNN
@@
 Connection ~ 7650 5900
 $Comp
-L GND #PWR0175
+L GND #PWR178
 U 1 1 58DDBCA6
 P 7900 5950
-F 0 "#PWR0175" H 8100 5850 50  0001 C CNN
+F 0 "#PWR178" H 8100 5850 50  0001 C CNN
 F 1 "GND" H 8100 5750 50  0001 C CNN
 F 2 "" H 7900 5950 50  0001 C CNN
@@
 $EndComp
 $Comp
-L GND #PWR0176
+L GND #PWR177
 U 1 1 58DDDADF
 P 7650 7050
-F 0 "#PWR0176" H 7850 6950 50  0001 C CNN
+F 0 "#PWR177" H 7850 6950 50  0001 C CNN
 F 1 "GND" H 7850 6850 50  0001 C CNN
 F 2 "" H 7650 7050 50  0001 C CNN
@@
 $EndComp
 $Comp
-L GND #PWR0177
+L GND #PWR172
 U 1 1 58DDDBB3
 P 6350 7050
-F 0 "#PWR0177" H 6550 6950 50  0001 C CNN
+F 0 "#PWR172" H 6550 6950 50  0001 C CNN
 F 1 "GND" H 6550 6850 50  0001 C CNN
 F 2 "" H 6350 7050 50  0001 C CNN
@@
 DVDDH
 $Comp
-L VCC_3.3V #PWR0178
+L VCC_3.3V #PWR160
 U 1 1 58E02074
 P 850 5250
-F 0 "#PWR0178" H 1030 5020 50  0001 C CNN
+F 0 "#PWR160" H 1030 5020 50  0001 C CNN
 F 1 "VCC_3.3V" H 980 5120 50  0001 C CNN
 F 2 "" H 850 5250 50  0001 C CNN
@@
 $EndComp
 $Comp
-L VCC_1.2V #PWR0179
+L VCC_1.2V #PWR161
 U 1 1 58E0210C
 P 850 6450
-F 0 "#PWR0179" H 1030 6220 50  0001 C CNN
+F 0 "#PWR161" H 1030 6220 50  0001 C CNN
 F 1 "VCC_1.2V" H 980 6320 50  0001 C CNN
 F 2 "" H 850 6450 50  0001 C CNN
@@
 $EndComp
 $Comp
-L VCC_3.3V #PWR0180
+L VCC_3.3V #PWR175
 U 1 1 58E021E4
 P 7550 3250
-F 0 "#PWR0180" H 7730 3020 50  0001 C CNN
+F 0 "#PWR175" H 7730 3020 50  0001 C CNN
 F 1 "VCC_3.3V" H 7680 3120 50  0001 C CNN
 F 2 "" H 7550 3250 50  0001 C CNN
@@
 Text GLabel 3250 3550 0    50   Input ~ 0
 PHY_MDINT
+Text Label 6100 3650 0    60   ~ 0
+phyad0
+Text Label 6100 3750 0    60   ~ 0
+phyad1
 $EndSCHEMATC

Commit message: footprints and footprint assignments
Parts:
- C176, C177, C182, C183, C184, C185, C186, C187, C218, C219, C221, C222, C223, C224, C227, C228, C250, C251, C252, C253, R100, R101, R102, R103, R104, R105, R106, R107, R108, R109, R110, R111, R112, R113, R114, R115, R116, R117, R118, R119, R120, R121, R122, R123, R124, R125, R51, R52, R95, R96, R97: footprint (none) -> footprints:0402
- C193, C216, C217, C220, C225, C226: footprint (none) -> footprints:0805
- FB1, FB2, FB3, R98, R99: footprint (none) -> footprints:0603
- J7: footprint (none) -> footprints:L829-1J1T-43
- TP22: footprint (none) -> footprints:TP_SMT
- U18: footprint (none) -> footprints:QFN48_EP_MICREL
- Y1: footprint (none) -> footprints:CTS_ATS

Commit message: add page titles to schematic
Other:
- note added: "Ethernet"
Changed lines of the file:
@@
 $Descr USLetter 11000 8500
 encoding utf-8
-Sheet 7 10
+Sheet 8 10
 Title ""
 Date ""
@@
 Text Label 6100 3750 0    60   ~ 0
 phyad1
+Text Notes 8900 900  0    150  ~ 30
+Ethernet
 $EndSCHEMATC
