File: kicad/firehose_08_power.sch (KiCad schematic (older format))
At the start: 0 parts

Commit message: more KiCAD schematic: power symbols, global nets
Parts:
- added C194, C198: 47 uF 20V, symbol CP
- added C195: 2.2 uF, symbol C
- added C196: 47 uF, symbol C
- added C197, C199: 0.1 uF 25V, symbol C
- added C200: 22 uF, symbol C
- added C213, C237: NONE, symbol C
- added J8: PJ-063BH, symbol PJ-063BH
- added L10: 0.47 uF, symbol L
- added L11: 1 uH, symbol L
- added LED4: LED, symbol LED
- added Q1: Si2369DS, symbol PMOSFET
- added R143, R145, R87: 0, symbol R
- added R70: 54.9k, symbol R
- added R71: 12.1k, symbol R
- added R72, R73: 10k, symbol R
- added R74: 162k, symbol R
- added R75: 330, symbol R
- added TP23, TP24, TP25, TP26: test_point, symbol test_point
- added U17: LTC3633, symbol LTC3633
- added Z1: SMAJ9.0CA, symbol TVS
Connections:
- net labels added: GND, VCC_1.2V, VCC_3.3V
- wire segments 0 -> 43

Commit message: footprints and footprint assignments
Parts:
- C194, C198: footprint (none) -> footprints:tantalum-size-D
- C195: footprint (none) -> footprints:0603
- C196, C200, C213, C237, R143, R87: footprint (none) -> footprints:1210
- C197, C199, R70, R71, R72, R73, R74, R75: footprint (none) -> footprints:0402
- J8: footprint (none) -> footprints:PJ-063BH
- L10, L11: footprint (none) -> footprints:NRS5020
- LED4: footprint (none) -> footprints:APA2106
- Q1: footprint (none) -> footprints:SOT23
- R145: footprint (none) -> footprints:0805
- TP23, TP24, TP25, TP26: footprint (none) -> footprints:TP_SMT
- U17: footprint (none) -> footprints:UFD28
- Z1: footprint (none) -> footprints:SMAJ

Commit message: add page titles to schematic
Other:
- note added: "1.2V"
- note added: "3.3V"
- note added: "5V"
- note added: "DC input"
- note added: "Power"
Changed lines of the file:
@@
 $Descr USLetter 11000 8500
 encoding utf-8
-Sheet 8 10
+Sheet 9 10
 Title ""
 Date ""
@@
 	1    0    0    -1
 $EndComp
+Text Notes 9050 950  0    150  ~ 30
+Power
+Text Notes 1050 3150 0    100  ~ 20
+DC input
+Text Notes 1250 3400 0    100  ~ 20
+5V
+Text Notes 2400 4650 0    100  ~ 20
+3.3V
+Text Notes 9600 4650 0    100  ~ 20
+1.2V
 $EndSCHEMATC
