File: kicad/firehose_09_mechanical.sch (KiCad schematic (older format))
At the start: 0 parts

Commit message: KiCAD schematic complete
Parts:
- added FID1, FID2, FID3: fiducial, symbol fiducial
- added MH1, MH2, MH3, MH4: mounting_hole, symbol mounting_hole
- added SC1, SC2, SC3, SC4, SC5, SC6, SC7, SC8: shield_clip, symbol shield_clip
Connections:
- net labels added: GND
Other:
- note added: "fiducials"
- note added: "mounting holes"
- note added: "shield clips for RF channels"

Commit message: footprints and footprint assignments
Parts:
- FID1, FID2, FID3: footprint (none) -> footprints:FIDUCIAL
- MH1, MH2, MH3, MH4: footprint (none) -> footprints:HOLE_UNC_2_56
- SC1, SC2, SC3, SC4, SC5, SC6, SC7, SC8: footprint (none) -> footprints:S1721
Changed lines of the file:
@@
 F 0 "SC1" H 2540 1200 60  0000 C CNN
 F 1 "shield_clip" H 2690 1080 60  0000 C CNN
-F 2 "" H 2350 1450 60  0001 C CNN
+F 2 "footprints:S1721" H 2350 1450 60  0001 C CNN
 F 3 "" H 2350 1450 60  0001 C CNN
 	1    2350 1450
@@
 F 0 "SC2" H 3690 1200 60  0000 C CNN
 F 1 "shield_clip" H 3840 1080 60  0000 C CNN
-F 2 "" H 3500 1450 60  0001 C CNN
+F 2 "footprints:S1721" H 3500 1450 60  0001 C CNN
 F 3 "" H 3500 1450 60  0001 C CNN
 	1    3500 1450
@@
 F 0 "SC3" H 2590 2100 60  0000 C CNN
 F 1 "shield_clip" H 2740 1980 60  0000 C CNN
-F 2 "" H 2400 2350 60  0001 C CNN
+F 2 "footprints:S1721" H 2400 2350 60  0001 C CNN
 F 3 "" H 2400 2350 60  0001 C CNN
 	1    2400 2350
@@
 F 0 "SC4" H 3690 2100 60  0000 C CNN
 F 1 "shield_clip" H 3840 1980 60  0000 C CNN
-F 2 "" H 3500 2350 60  0001 C CNN
+F 2 "footprints:S1721" H 3500 2350 60  0001 C CNN
 F 3 "" H 3500 2350 60  0001 C CNN
 	1    3500 2350
@@
 F 0 "SC5" H 2590 3050 60  0000 C CNN
 F 1 "shield_clip" H 2740 2930 60  0000 C CNN
-F 2 "" H 2400 3300 60  0001 C CNN
+F 2 "footprints:S1721" H 2400 3300 60  0001 C CNN
 F 3 "" H 2400 3300 60  0001 C CNN
 	1    2400 3300
@@
 F 0 "SC6" H 3690 3000 60  0000 C CNN
 F 1 "shield_clip" H 3840 2880 60  0000 C CNN
-F 2 "" H 3500 3250 60  0001 C CNN
+F 2 "footprints:S1721" H 3500 3250 60  0001 C CNN
 F 3 "" H 3500 3250 60  0001 C CNN
 	1    3500 3250
@@
 F 0 "SC7" H 2590 3950 60  0000 C CNN
 F 1 "shield_clip" H 2740 3830 60  0000 C CNN
-F 2 "" H 2400 4200 60  0001 C CNN
+F 2 "footprints:S1721" H 2400 4200 60  0001 C CNN
 F 3 "" H 2400 4200 60  0001 C CNN
 	1    2400 4200
@@
 F 0 "SC8" H 3740 3950 60  0000 C CNN
 F 1 "shield_clip" H 3890 3830 60  0000 C CNN
-F 2 "" H 3550 4200 60  0001 C CNN
+F 2 "footprints:S1721" H 3550 4200 60  0001 C CNN
 F 3 "" H 3550 4200 60  0001 C CNN
 	1    3550 4200
@@
 F 0 "FID1" H 2210 5920 60  0000 C CNN
 F 1 "fiducial" H 2280 5820 60  0000 C CNN
-F 2 "" H 2000 6200 60  0001 C CNN
+F 2 "footprints:FIDUCIAL" H 2000 6200 60  0001 C CNN
 F 3 "" H 2000 6200 60  0001 C CNN
 	1    2000 6200
@@
 F 0 "FID2" H 3410 5920 60  0000 C CNN
 F 1 "fiducial" H 3480 5820 60  0000 C CNN
-F 2 "" H 3200 6200 60  0001 C CNN
+F 2 "footprints:FIDUCIAL" H 3200 6200 60  0001 C CNN
 F 3 "" H 3200 6200 60  0001 C CNN
 	1    3200 6200
@@
 F 0 "FID3" H 4560 5920 60  0000 C CNN
 F 1 "fiducial" H 4630 5820 60  0000 C CNN
-F 2 "" H 4350 6200 60  0001 C CNN
+F 2 "footprints:FIDUCIAL" H 4350 6200 60  0001 C CNN
 F 3 "" H 4350 6200 60  0001 C CNN
 	1    4350 6200
@@
 F 0 "MH1" H 7120 1760 60  0000 C CNN
 F 1 "mounting_hole" H 7230 1670 60  0000 C CNN
-F 2 "" H 6800 2100 60  0001 C CNN
+F 2 "footprints:HOLE_UNC_2_56" H 6800 2100 60  0001 C CNN
 F 3 "" H 6800 2100 60  0001 C CNN
 	1    6800 2100
@@
 F 0 "MH2" H 8520 1760 60  0000 C CNN
 F 1 "mounting_hole" H 8630 1670 60  0000 C CNN
-F 2 "" H 8200 2100 60  0001 C CNN
+F 2 "footprints:HOLE_UNC_2_56" H 8200 2100 60  0001 C CNN
 F 3 "" H 8200 2100 60  0001 C CNN
 	1    8200 2100
@@
 F 0 "MH3" H 7120 3060 60  0000 C CNN
 F 1 "mounting_hole" H 7230 2970 60  0000 C CNN
-F 2 "" H 6800 3400 60  0001 C CNN
+F 2 "footprints:HOLE_UNC_2_56" H 6800 3400 60  0001 C CNN
 F 3 "" H 6800 3400 60  0001 C CNN
 	1    6800 3400
@@
 F 0 "MH4" H 8570 3060 60  0000 C CNN
 F 1 "mounting_hole" H 8680 2970 60  0000 C CNN
-F 2 "" H 8250 3400 60  0001 C CNN
+F 2 "footprints:HOLE_UNC_2_56" H 8250 3400 60  0001 C CNN
 F 3 "" H 8250 3400 60  0001 C CNN
 	1    8250 3400
@@
 fiducials
 $Comp
-L GND #PWR207
+L GND #PWR0199
 U 1 1 58DEE757
 P 6800 2650
-F 0 "#PWR207" H 7000 2550 50  0001 C CNN
+F 0 "#PWR0199" H 7000 2550 50  0001 C CNN
 F 1 "GND" H 7000 2450 50  0001 C CNN
 F 2 "" H 6800 2650 50  0001 C CNN
@@
 $EndComp
 $Comp
-L GND #PWR209
+L GND #PWR0200
 U 1 1 58DEE7CD
 P 8200 2650
-F 0 "#PWR209" H 8400 2550 50  0001 C CNN
+F 0 "#PWR0200" H 8400 2550 50  0001 C CNN
 F 1 "GND" H 8400 2450 50  0001 C CNN
 F 2 "" H 8200 2650 50  0001 C CNN
@@
 $EndComp
 $Comp
-L GND #PWR210
+L GND #PWR0201
 U 1 1 58DEE85B
 P 8250 3950
-F 0 "#PWR210" H 8450 3850 50  0001 C CNN
+F 0 "#PWR0201" H 8450 3850 50  0001 C CNN
 F 1 "GND" H 8450 3750 50  0001 C CNN
 F 2 "" H 8250 3950 50  0001 C CNN
@@
 $EndComp
 $Comp
-L GND #PWR208
+L GND #PWR0202
 U 1 1 58DEE8B1
 P 6800 3950
-F 0 "#PWR208" H 7000 3850 50  0001 C CNN
+F 0 "#PWR0202" H 7000 3850 50  0001 C CNN
 F 1 "GND" H 7000 3750 50  0001 C CNN
 F 2 "" H 6800 3950 50  0001 C CNN
@@
 $EndComp
 $Comp
-L GND #PWR199
+L GND #PWR0203
 U 1 1 58DEE961
 P 2350 1700
-F 0 "#PWR199" H 2550 1600 50  0001 C CNN
+F 0 "#PWR0203" H 2550 1600 50  0001 C CNN
 F 1 "GND" H 2550 1500 50  0001 C CNN
 F 2 "" H 2350 1700 50  0001 C CNN
@@
 $EndComp
 $Comp
-L GND #PWR203
+L GND #PWR0204
 U 1 1 58DEE999
 P 3500 1700
-F 0 "#PWR203" H 3700 1600 50  0001 C CNN
+F 0 "#PWR0204" H 3700 1600 50  0001 C CNN
 F 1 "GND" H 3700 1500 50  0001 C CNN
 F 2 "" H 3500 1700 50  0001 C CNN
@@
 $EndComp
 $Comp
-L GND #PWR200
+L GND #PWR0205
 U 1 1 58DEE9D1
 P 2400 2600
-F 0 "#PWR200" H 2600 2500 50  0001 C CNN
+F 0 "#PWR0205" H 2600 2500 50  0001 C CNN
 F 1 "GND" H 2600 2400 50  0001 C CNN
 F 2 "" H 2400 2600 50  0001 C CNN
@@
 $EndComp
 $Comp
-L GND #PWR204
+L GND #PWR0206
 U 1 1 58DEEA09
 P 3500 2600
-F 0 "#PWR204" H 3700 2500 50  0001 C CNN
+F 0 "#PWR0206" H 3700 2500 50  0001 C CNN
 F 1 "GND" H 3700 2400 50  0001 C CNN
 F 2 "" H 3500 2600 50  0001 C CNN
@@
 $EndComp
 $Comp
-L GND #PWR201
+L GND #PWR0207
 U 1 1 58DEEA41
 P 2400 3550
-F 0 "#PWR201" H 2600 3450 50  0001 C CNN
+F 0 "#PWR0207" H 2600 3450 50  0001 C CNN
 F 1 "GND" H 2600 3350 50  0001 C CNN
 F 2 "" H 2400 3550 50  0001 C CNN
@@
 $EndComp
 $Comp
-L GND #PWR205
+L GND #PWR0208
 U 1 1 58DEEA79
 P 3500 3500
-F 0 "#PWR205" H 3700 3400 50  0001 C CNN
+F 0 "#PWR0208" H 3700 3400 50  0001 C CNN
 F 1 "GND" H 3700 3300 50  0001 C CNN
 F 2 "" H 3500 3500 50  0001 C CNN
@@
 $EndComp
 $Comp
-L GND #PWR202
+L GND #PWR0209
 U 1 1 58DEEAB1
 P 2400 4450
-F 0 "#PWR202" H 2600 4350 50  0001 C CNN
+F 0 "#PWR0209" H 2600 4350 50  0001 C CNN
 F 1 "GND" H 2600 4250 50  0001 C CNN
 F 2 "" H 2400 4450 50  0001 C CNN
@@
 $EndComp
 $Comp
-L GND #PWR206
+L GND #PWR0210
 U 1 1 58DEEAE9
 P 3550 4450
-F 0 "#PWR206" H 3750 4350 50  0001 C CNN
+F 0 "#PWR0210" H 3750 4350 50  0001 C CNN
 F 1 "GND" H 3750 4250 50  0001 C CNN
 F 2 "" H 3550 4450 50  0001 C CNN

Commit message: add page titles to schematic
Other:
- note added: "Mechanical"
Changed lines of the file:
@@
 $Descr USLetter 11000 8500
 encoding utf-8
-Sheet 9 10
+Sheet 10 10
 Title ""
 Date ""
@@
 	1    0    0    -1
 $EndComp
+Text Notes 8600 950  0    150  ~ 30
+Mechanical
 $EndSCHEMATC
